File: usb-dac.kicad_pcb (KiCad board)
At the start: 2 copper layers, 1.4 x 13 mm, 28 parts, among them J1 USB_C_Receptacle_USB2.0_14P, J2 AudioJack3, U1 PCM2912APJTR, Y1 6 MHz

Commit message: Finish PCB and clarify schematic
Parts:
- moved C4 42.3 mm to (123.3, 101.5), turned to -90 degrees
- moved C5 36.6 mm to (128.7, 101.5), turned to -90 degrees
- moved C6 31.2 mm to (134.0, 101.5), turned to -90 degrees
- moved C1 20.8 mm to (124.0, 90.5)
- moved J1 14.0 mm to (101.1, 94.5)
- moved L1 13.1 mm to (111.4, 99.4)
- moved R1 13.1 mm to (110.4, 78.4)
- moved R3 13.1 mm to (110.4, 94.3)
- moved R2 13.1 mm to (110.4, 89.0)
- moved R9 13.1 mm to (110.4, 83.7)
- moved C7 10.6 mm to (139.4, 101.5)
- moved J2 10.5 mm to (176.0, 94.5)
- moved C8 9.50 mm to (144.8, 101.5)
- moved R8 7.85 mm to (164.7, 92.0)
- moved R6 7.85 mm to (164.7, 95.9)
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Routing:
- net GND: track 0.00 -> 212.2 mm
- net /XTO: track 0.00 -> 41.1 mm
- net /VCCL: track 0.00 -> 32.1 mm
- net VBUS: track 0.00 -> 29.7 mm
- net /XTI: track 0.00 -> 28.4 mm
- net Net-(U1-VBUS): track 0.00 -> 24.1 mm
- net Net-(J1-D--PadA7): track 0.00 -> 22.1 mm
- net /VOUTL: track 0.00 -> 21.4 mm
- net /VOUTR: track 0.00 -> 21.1 mm
- net Net-(C10-Pad2): track 0.00 -> 17.9 mm
- net /D-: track 0.00 -> 17.3 mm
- net Net-(J1-CC1): track 0.00 -> 17.1 mm
- net Net-(C9-Pad2): track 0.00 -> 16.8 mm
- net Net-(J1-D+-PadA6): track 0.00 -> 12.7 mm
- net /VCCA: track 0.00 -> 12.5 mm
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- added copper zone on B.Cu, net GND
- added copper zone on F.Cu, net GND
Other:
- board size 1.4 x 13 mm -> 82.5 x 39 mm
