File: usb-dac.kicad_pcb (KiCad board)
At the start: 2 copper layers, 82.5 x 39 mm, 28 parts, among them J1 USB_C_Receptacle_USB2.0_14P, J2 AudioJack3, U1 PCM2912APJTR, Y1 6 MHz

Commit message: add "branding"
Other:
- board text added: "WhatWare USB DAC"
Changed lines of the file:
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@@
 		(layer "Edge.Cuts")
+	)
+	(gr_text "WhatWare\nUSB DAC"
+		(at 173 82.5 0)
+		(layer "F.SilkS")
+		(effects
+			(font
+				(size 1 1)
+				(thickness 0.1)
+			)
+			(justify bottom)
+		)
 	)
 	(segment
